File: Esquema_Mod_ReleFarol/Esquema_ReleFarol.kicad_pcb (KiCad board)
At the start: 2 copper layers, 0 parts

Commit message: [ADD] some projects
Parts:
- added F1: F3A 250V, Fuse:Fuseholder_Clip-5x20mm_Littelfuse_519_Inline_P20.60x5.00mm_D1.00mm_Horizontal, F.Cu at (145.2, 79.8)
- added J1: Conn_01x02_Socket, Connector_AMASS:AMASS_XT60PW-F_1x02_P7.20mm_Horizontal, F.Cu at (165.9, 86.8)
- added J2: Conn_01x02_Pin, Connector_AMASS:AMASS_XT60PW-M_1x02_P7.20mm_Horizontal, F.Cu at (155.8, 86.8)
- added J3: Servo CUAV A8, Connector_PinHeader_1.00mm:PinHeader_1x03_P1.00mm_Horizontal, F.Cu at (176.4, 71.5)
- added K1: HF41F, Relay_THT:Relay_SPDT_Finder_34.51_Vertical, F.Cu at (167.6, 73.5)
- added U1: 817B, Package_DIP:DIP-4_W7.62mm, F.Cu at (168.7, 78.5)
Routing:
- net (no net): vias 16 -> 0
Other:
- board text removed: "Anode"
- board text removed: "C"
- board text removed: "Cathode"
- board text removed: "E"
- board text removed: "F1"
- board text removed: "J1+"
- board text removed: "J2+"
- board text removed: "K1"
- board text removed: "M1 PWM"
- board text removed: "M1+"
- board text removed: "M1-"
- board text removed: "U1"
