File: Esquema_Mod_ReleFarol/Esquema_ReleFarol.kicad_sch (KiCad schematic)
At the start: 6 parts, among them J1 Conn_01x02_Socket, J2 Conn_01x02_Pin, K1 G6E, M1 Motor_Servo, U1 LTV-817

Commit message: [ADD] some projects
Parts:
- removed M1: Motor_Servo, symbol Motor:Motor_Servo
- added J3: Servo CUAV A8, Connector_PinHeader_1.00mm:PinHeader_1x03_P1.00mm_Horizontal, symbol Connector:Conn_01x03_Socket
- F1: value Fuse -> F3A 250V; footprint (none) -> Fuse:Fuseholder_Clip-5x20mm_Littelfuse_519_Inline_P20.60x5.00mm_D1.00mm_Horizontal
- J1: footprint (none) -> Connector_AMASS:AMASS_XT60PW-F_1x02_P7.20mm_Horizontal
- J2: footprint (none) -> Connector_AMASS:AMASS_XT60PW-M_1x02_P7.20mm_Horizontal
- K1: value G6E -> HF41F; footprint Relay_THT:Relay_SPDT_Omron_G6E -> Relay_THT:Relay_SPDT_Finder_34.51_Vertical
- U1: value LTV-817 -> 817B
Connections:
- net at U1.1: now also J3.3 (Pin_3)
- net at K1.1: now also J3.2 (Pin_2)
- net at U1.2, U1.3: now also J3.1 (Pin_1)
- no-connect marks 0 -> 1
Other:
- note removed: "817B"
- note removed: "HF41F"
- company: (none) -> SkyDrones
- title: (none) -> Driver Farol
- moved on the sheet: F1, J1, J2, K1
