File: Esquema_Mod_Buzzer/Esquema_Buzzer.kicad_sch (KiCad schematic)
At the start: 12 parts, among them J1 XT30-M, M1 Motor_Servo, Q1 BC337, U1 817B, U2 MT3608, U3 MT3608

Commit message: [ADD]
Parts:
- removed M1: Motor_Servo, symbol Motor:Motor_Servo
- removed U1: 817B, Package_DIP:DIP-4_W7.62mm, symbol Isolator:LTV-817
- removed U3: MT3608, Package_TO_SOT_SMD:SOT-23-6, symbol Regulator_Switching:MT3608
- added D1: SS34, Diode_SMD:D_2114_3652Metric_Pad1.85x3.75mm_HandSolder, symbol Device:D
- added J2: Conn_01x03_Pin, Connector_PinHeader_1.00mm:PinHeader_1x03_P1.00mm_Horizontal, symbol Connector:Conn_01x03_Pin
- added L1: 10uH, Inductor_SMD:L_7.3x7.3_H4.5, symbol Device:L
- added U1: PC817, Package_DIP:DIP-4_W7.62mm, symbol Isolator:PC817
- BZ1: footprint (none) -> Buzzer_Beeper:Buzzer_12x9.5RM7.6
- C1: value C -> 100uf; footprint (none) -> Capacitor_SMD:CP_Elec_3x5.3
- C2: value C -> 22uF; footprint (none) -> Capacitor_SMD:CP_Elec_3x5.3
- J1: value XT30-M -> Conn_01x02_Pin; footprint (none) -> Connector_AMASS2:AMASS_XT30PW-M_1x02_P2.50mm_Horizontal
- R1: footprint (none) -> Resistor_THT:R_Axial_DIN0204_L3.6mm_D1.6mm_P5.08mm_Horizontal
- R2: value R -> 10k; footprint (none) -> Resistor_SMD:R_0201_0603Metric
- R3: value R -> 390; footprint (none) -> Resistor_SMD:R_0201_0603Metric
Connections:
- net at BZ1.2 (-), Q1.1 (C): now also R1.1; no longer R1.2
- net at Q1.2 (B): now also U1.3
- net at U2.4 (EN): now also C2.1, J1.2 (Pin_2), U2.5 (IN), L1.1, U1.4; no longer Q1.3 (E)
- net at U2.1 (SW): now also D1.2 (A), L1.2; no longer J1.2 (Pin_2)
- net GND: now reaches J1.1 (Pin_1), U2.2 (GND)
- net GND: now also C1.2, C2.2, Q1.3 (E), R3.1
- net at R2.1: now also R3.2, U2.3 (FB)
- net at R2.2: now also BZ1.1 (+), C1.1, R1.2, D1.1 (K)
- new net: J2.3 (Pin_3), U1.1
- new net: J2.1 (Pin_1), U1.2
- no-connect marks 0 -> 1
Other:
- company: (none) -> SkyDrones
- title: (none) -> Placa Buzzer
- moved on the sheet: BZ1, Q1, R1

Commit message: [ADD] some projects
Parts:
- J1: footprint Connector_AMASS2:AMASS_XT30PW-M_1x02_P2.50mm_Horizontal -> Amass:AMASS_XT30PW-M_1x02_P2.50mm_Horizontal
Other:
- title: Placa Buzzer -> Módulo Buzzer
Changed lines of the file:
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@@
 	(paper "A4")
 	(title_block
-		(title "Placa Buzzer")
-		(date "2026-02-10")
+		(title "Módulo Buzzer")
+		(date "2026-02-25")
+		(rev "2.0")
 		(company "SkyDrones")
+		(comment 1 "Drawn by Murillo S. Horvath")
 	)
 	(junction
@@
 			)
 		)
-		(property "Footprint" "Connector_AMASS2:AMASS_XT30PW-M_1x02_P2.50mm_Horizontal"
+		(property "Footprint" "Amass:AMASS_XT30PW-M_1x02_P2.50mm_Horizontal"
 			(at 87.63 78.74 0)
 			(effects

Commit message: [UP] Upgrade Buzzer
Parts:
- J2: footprint Connector_PinHeader_1.00mm:PinHeader_1x03_P1.00mm_Horizontal -> Connector_PinHeader_2.54mm:PinHeader_1x03_P2.54mm_Horizontal
- R2: value 10k -> 90k
- R3: value 390 -> 2.2k
Other:
- moved on the sheet: R2
Changed lines of the file:
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@@
-	)
-	(junction
-		(at 171.45 97.79)
-		(diameter 0)
-		(color 0 0 0 0)
 	)
 	(junction
@@
 	)
 	(junction
+		(at 171.45 93.98)
+		(diameter 0)
+		(color 0 0 0 0)
+	)
+	(junction
 		(at 114.3 76.2)
 		(diameter 0)
@@
 	(wire
 		(pts
-			(xy 171.45 85.09) (xy 171.45 76.2)
+			(xy 171.45 81.28) (xy 171.45 76.2)
 		)
 		(stroke
@@
 	(wire
 		(pts
-			(xy 146.05 93.98) (xy 157.48 93.98)
+			(xy 146.05 93.98) (xy 171.45 93.98)
 		)
 		(stroke
@@
 	(wire
 		(pts
-			(xy 157.48 93.98) (xy 157.48 97.79)
-		)
-		(stroke
-			(width 0)
-			(type default)
-		)
-	)
-	(wire
-		(pts
 			(xy 184.15 92.71) (xy 184.15 113.03)
 		)
@@
 	(wire
 		(pts
-			(xy 171.45 97.79) (xy 171.45 100.33)
+			(xy 171.45 93.98) (xy 171.45 100.33)
 		)
 		(stroke
@@
 	(wire
 		(pts
-			(xy 157.48 97.79) (xy 171.45 97.79)
-		)
-		(stroke
-			(width 0)
-			(type default)
-		)
-	)
-	(wire
-		(pts
 			(xy 121.92 88.9) (xy 130.81 88.9)
 		)
@@
 	(wire
 		(pts
-			(xy 171.45 92.71) (xy 171.45 97.79)
+			(xy 171.45 88.9) (xy 171.45 93.98)
 		)
 		(stroke
@@
 			)
 		)
-		(property "Value" "390"
+		(property "Value" "2.2k"
 			(at 176.784 103.378 0)
 			(effects
@@
 	(symbol
 		(lib_id "Device:R")
-		(at 171.45 88.9 180)
+		(at 171.45 85.09 180)
 		(unit 1)
 		(exclude_from_sim no)
@@
 		(dnp no)
 		(property "Reference" "R2"
-			(at 175.768 90.424 0)
-			(effects
-				(font
-					(size 1.27 1.27)
-				)
-				(justify left)
-			)
-		)
-		(property "Value" "10k"
-			(at 176.53 87.884 0)
+			(at 175.768 86.614 0)
+			(effects
+				(font
+					(size 1.27 1.27)
+				)
+				(justify left)
+			)
+		)
+		(property "Value" "90k"
+			(at 176.53 84.074 0)
 			(effects
 				(font
@@
 		)
 		(property "Footprint" "Resistor_SMD:R_0201_0603Metric"
-			(at 173.228 88.9 90)
+			(at 173.228 85.09 90)
 			(effects
 				(font
@@
 		)
 		(property "Datasheet" "~"
-			(at 171.45 88.9 0)
+			(at 171.45 85.09 0)
 			(effects
 				(font
@@
 		)
 		(property "Description" "Resistor"
-			(at 171.45 88.9 0)
+			(at 171.45 85.09 0)
 			(effects
 				(font
@@
 			)
 		)
-		(property "Footprint" "Connector_PinHeader_1.00mm:PinHeader_1x03_P1.00mm_Horizontal"
+		(property "Footprint" "Connector_PinHeader_2.54mm:PinHeader_1x03_P2.54mm_Horizontal"
 			(at 88.9 102.87 0)
 			(effects
