File: Personal-Projects/09_Esquema_Mod_STM32gpsTracker/Esquema_Mod_STM32gpsTracker.kicad_sch (KiCad schematic)
At the start: 55 parts, among them J1 Screw_Terminal_01x02, J2 693010020611, J3 RIGHT HEADER PINS, J4 LEFT HEADER PINS, Q1 AO3407A, SW1 SW_Push, SW2 SW_Push, U1 TPS5430DDA, U2 STM32F030C8Tx, U3 SMF05CT1G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

Commit message: [ADD] project 09
Parts:
- added C19: 4u7, symbol Device:C
- added R13: 4K7, symbol Device:R
- Q1: footprint SOT95P280X125-3N -> LIB_AO3407A:SOT95P280X125-3N
Connections:
- net GND: now also C19.1
- net SIM_CLK: now also U4.31 (SIM_CLK)
- net SIM_DATA: now also U4.30 (SIM_DATA)
- net SIM_DET: now also U4.33 (SIM_DET), R13.2
- net SIM_RST: now also U4.32 (SIM_RST)
- net SIM_VDD: now also U4.29 (SIM_VDD)
- net STATUS: now also U4.49 (STATUS)
- net at U4.17 (VRTC): now also C19.2
- net GPS_ANT: now reaches U4.35 (GPS_ANT)
- net GPS_ANT: now also U4.66 (GSM_ANT)
- net at U4.7 (VDD_EXT): now also R13.1
- no-connect marks 47 -> 63
Other:
- note added: "SIM808"
