File: Personal-Projects/09_Esquema_Mod_STM32gpsTracker/Esquema_Mod_STM32gpsTracker.kicad_sch (KiCad schematic)
At the start: 57 parts, among them J1 Screw_Terminal_01x02, J2 693010020611, J3 RIGHT HEADER PINS, J4 LEFT HEADER PINS, Q1 AO3407A, SW1 SW_Push, SW2 SW_Push, U1 TPS5430DDA, U2 STM32F030C8Tx, U3 SMF05CT1G, U4 SIM808, Y1 Crystal

Commit message: [ADD] New Project
FPV Drone new project hardware
Parts:
- C1: footprint (none) -> Capacitor_SMD:C_0805_2012Metric
- C10, C11, C12, C13, C14, C5, C6, C7, C8, C9: footprint (none) -> Capacitor_SMD:C_0402_1005Metric
- C15: value C -> 1uF; footprint (none) -> Capacitor_SMD:C_0402_1005Metric
- C16: value C -> 100uF; footprint (none) -> Capacitor_SMD:C_1206_3216Metric
- C17: value C -> 33pF; footprint (none) -> Capacitor_SMD:C_0402_1005Metric
- C18: value C -> 10pF; footprint (none) -> Capacitor_SMD:C_0402_1005Metric
- C19: footprint (none) -> Capacitor_SMD:C_0603_1608Metric
- C2, C4: footprint (none) -> Capacitor_SMD:C_0201_0603Metric
- C3: footprint (none) -> Capacitor_Tantalum_SMD:CP_EIA-7343-15_Kemet-W
Connections:
- net PA7/SPI_MOSI is gone; now on net PA7/SPI1_MOSI: J4.2 (Pin_2)
- net USART_RX is gone; now on net USART2_RX: J4.6 (Pin_6)
