File: SkyDrones-Projects/FPV-Drone-Hardware/1-FlightController/Schematics/1-FlightController.kicad_sch (KiCad schematic)
At the start: 4 parts, among them U1 STM32F405RGTx, U2 MPU-6000, U3 BMP280, U4 W25Q128JVS

Commit message: Some Projects
Parts:
- removed U1: STM32F405RGTx, Package_QFP:LQFP-64_10x10mm_P0.5mm, symbol MCU_ST_STM32F4:STM32F405RGTx
- removed U2: MPU-6000, MPU-6000:QFN-24, symbol MPU-6000:MPU-6000
- removed U3: BMP280, Package_LGA:Bosch_LGA-8_2x2.5mm_P0.65mm_ClockwisePinNumbering, symbol Sensor_Pressure:BMP280
- removed U4: W25Q128JVS, Package_SON:WSON-8-1EP_8x6mm_P1.27mm_EP3.4x4.3mm, symbol Memory_Flash:W25Q128JVS
- added C1: 4.7uF, Capacitor_SMD:C_0805_2012Metric, symbol Device:C
- added C10, C8: 1uF, Capacitor_SMD:C_0603_1608Metric, symbol Device:C
- added C11, C9: 2.2uF, Capacitor_SMD:C_0603_1608Metric, symbol Device:C
- added C12: 2.2uF, symbol Device:C
- added C13, C14, C15, C16, C17, C18, C21, C23, C24: 100nF, symbol Device:C
- added C19, C20: 22pF, symbol Device:C
- added C2: 100nF, Capacitor_SMD:C_0603_1608Metric, symbol Device:C
- added C22: 2.2Uf, symbol Device:C
- added C3, C4, C5, C6, C7: 47uF, Capacitor_SMD:C_0805_2012Metric, symbol Device:C
- added D1, D2, D5: 16-213/GHC-YR1S2/3T, LED_SMD:LED_0402_1005Metric, symbol Device:LED
- added D3, D4: 1N5819WS, Diode_SMD:D_SOD-323, symbol Diode:1N5819WS
- added J1: USB_C_Receptacle, symbol Connector:USB_C_Receptacle
- added R1: 10k, Resistor_SMD:R_0603_1608Metric, symbol Device:R
- added R2: 75k, Resistor_SMD:R_0603_1608Metric, symbol Device:R
- added R3: 14k3, Resistor_SMD:R_0603_1608Metric, symbol Device:R
- added R4, R7: 1k, Resistor_SMD:R_0603_1608Metric, symbol Device:R
- added R5, R6: 100k, Resistor_SMD:R_0603_1608Metric, symbol Device:R
- added R8: 10k, symbol Device:R
- added R9: R, symbol Device:R
- added U1, U2: ZL6205A33TS5, Package_TO_SOT_SMD:SOT-23-5, symbol Regulator_Linear:AP2112K-3.3
- added U3: STM32F405RGTx, Package_QFP:LQFP-64_10x10mm_P0.5mm, symbol MCU_ST_STM32F4:STM32F405RGTx
- added U4: MPU-6000, MPU-6000:QFN-24, symbol MPU-6000:MPU-6000
- added U5: MPM3550EGLE, Package_LGA:MPS_LGA-18-10EP_12x12mm_P3.3mm, symbol Regulator_Switching:MPM3550EGLE
- added U6: BMP280, Package_LGA:Bosch_LGA-8_2x2.5mm_P0.65mm_ClockwisePinNumbering, symbol Sensor_Pressure:BMP280
- added U7: USBLC6-2SC6, Package_TO_SOT_SMD:SOT-23-6, symbol Power_Protection:USBLC6-2SC6
- added U8: W25Q128JVP, Package_SON:WSON-8-1EP_6x5mm_P1.27mm_EP3.4x4.3mm, symbol Memory_Flash:W25Q128JVP
- added Y1: 8MHz, symbol Device:Crystal
Connections:
- new net: D2.1 (K), R4.1
- new net: R6.2, U5.2 (RFREQ)
- new net: D1.1 (K), R1.1
- new net: R5.2, U5.1 (EN)
- new net: R2.2, R3.1, U5.4 (FB)
- new net: D5.1 (K), R7.1
- new net: C18.1, R8.2, U3.60 (BOOT0), U3.7 (NRST)
- new net: J1.A1 (GND), J1.A12 (GND), J1.B1 (GND), J1.B12 (GND)
- new net: J1.A4 (VBUS), J1.A9 (VBUS), J1.B4 (VBUS), J1.B9 (VBUS)
- new net: C22.1, U4.20 (CPOUT)
- new net: C20.2, U3.5 (PH0), Y1.2
- new net: C19.2, U3.6 (PH1), Y1.1
- new net 3V3: C12.1, C13.1, C14.1, C15.1, C16.1, C17.1, C23.1, C24.1, C9.1, D5.2 (A), R8.1, U1.5 (VOUT), U3.1 (VBAT), U3.13 (VDDA), U3.19 (VDD), U3.32 (VDD), U3.48 (VDD), U3.64 (VDD), U6.6 (VDDIO), U6.8 (VDD)
- new net 3V3_MPU: C11.1, C21.1, U2.5 (VOUT), U4.13 (VDD)
- new net 5V: C10.1, C8.1, D3.1 (K), D4.1 (K), U1.1 (VIN), U1.3 (EN), U2.1 (VIN), U2.3 (EN)
- new net 5VREG: C3.1, C4.1, C5.1, C6.1, C7.1, D2.2 (A), D4.2 (A), R2.1, U5.5 (VOUT)
- new net 5VUSB: D3.2 (A)
- new net GND: C1.2, C10.2, C11.2, C12.2, C13.2, C14.2, C15.2, C16.2, C17.2, C18.2, C19.1, C2.2, C20.1, C21.2, C22.2, C23.2, C24.2, C3.2, C4.2, C5.2, C6.2, C7.2, C8.2, C9.2, R1.2, R3.2, R4.2, R6.1, R7.2, U1.2 (GND), U2.2 (GND), U3.12 (VSSA), U3.18 (VSS), U3.63 (VSS), U4.1 (CLKIN), U4.18 (GND), U5.10 (GND), U5.11 (GND), U5.12 (GND), U5.13 (GND), U5.14 (GND), U5.15 (GND), U5.16 (GND), U5.17 (GND), U5.18 (GND), U5.6 (GND), U5.7 (GND), U5.9 (GND), U6.1 (GND), U6.7 (GND)
- new net SPI_CS1: U4.8 (/CS)
- new net SPI_MISO1: U4.9 (AD0/SDO)
- new net SPI_MOSI1: U4.24 (SDA/SDI)
- new net VBAT: C1.1, C2.1, D1.2 (A), R5.1, U5.8 (VIN)
- no-connect marks 0 -> 11
Other:
- note added: "Alimentação Buck 5V"
- note added: "Alimentação LDO 3.3V"
- note added: "Baro BMP280"
- note added: "Gyro MPU6000"
- note added: "MCU"
