File: Empresa-EcoQuali/EC01/outputs/EC01_KiCad_REV0_2/KiCad/01_Alimentacao_Bateria.kicad_sch (KiCad schematic)
At the start: 21 parts, among them Q1 AO3401A, SW1 CHAVE GERAL, U1 TPS63802DLAR

Commit message: EC01
Connections:
- net BAT_SW: now also SW1.1 (IN); no longer SW1.2 (OUT)
- net BAT_FUSED: no longer names the net of F1.2, Q1.3 (D)
- net BAT_PROT: no longer names the net of Q1.2 (S)
- net BAT_PROT: now also SW1.2 (OUT); no longer SW1.1 (IN)
- net BAT_RAW: no longer names the net of BT1.1 (+), F1.1
- net PSU_FB: no longer names the net of R1.2, R2.1, U1.4 (FB)
- net SW_L1: no longer names the net of L1.1, U1.9 (L1)
- net SW_L2: no longer names the net of L1.2, U1.7 (L2)
Other:
- note added: "ADC: 100k/100k e C5=100nF mantidos. Opcao 1M/1M depende de fuga e tempo de acomodacao."
- note added: "EN: R3/R4 = 200k/100k. Corte nominal 3,30 V / 3,00 V; conferir tolerancias."
- note removed: "Celula 1S protegida e removivel. Sem carregador. USB nao alimenta o circuito."
- note removed: "F1, F2, suporte e chave exigem selecao mecanica e coordenacao de protecao."
- note removed: "TPS63802: 3,308 V nominal. EN: liga em ~3,30 V; desliga em ~3,00 V."
- moved on the sheet: BT1, C1, C2, C3, C4, C5, F1, L1, Q1, R1, R2, R3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
