File: Empresa-EcoQuali/EC01/outputs/EC01_KiCad_REV0_2/KiCad/02_ESP32_Inicializacao.kicad_sch (KiCad schematic)
At the start: 21 parts, among them SW2 RESET SPST-NO, SW3 BOOT SPST-NO, U2 ESP32-C3FH4

Commit message: EC01
Parts:
- L2: value 24nH >=500mA -> FILTRO RF TBD >=500mA; Decisao Filtro ALIMENTACAO, nunca conectar a LNA_IN. Valor inicial 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 -> Valor 24nH removido: recomendacao de 24nH pertence ao XTAL_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
Other:
- note added: "L2: valor/MPN do filtro de alimentacao RF pendentes. 24nH aplica-se ao XTAL_P (folha 03)."
- moved on the sheet: C10, C11, C12, C13, C6, C7, C8, C9, L2, R10, R11, R12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
