File: Empresa-EcoQuali/EC01/outputs/EC01_KiCad_REV0_2/KiCad/03_BLE_Cristal.kicad_sch (KiCad schematic)
At the start: 10 parts, among them Y1 40MHz CL=8pF <=10ppm

Commit message: EC01
Parts:
- added L4: 24nH TUNE, symbol EC01:EC01_L4
Connections:
- net XTAL_P: now also L4.1; no longer C14.1, Y1.1 (X1)
- net BLE_50R: no longer names the net of C17.1, C18.1, L3.2, R14.1
- net BLE_ANT: no longer names the net of ANT1.1 (FEED), C19.1, R14.2
- new net: C14.1, L4.2, Y1.1 (X1)
Other:
- note added: "L4=24nH e C14/C15=10pF sao pontos de partida; CL=8pF pressupoe cerca de 3pF parasitas."
- note added: "LNA_IN sem ligacao DC ao 3V3. Rede CLC e IFA exigem ajuste de RF e geometria de PCB."
- note added: "OSCILADOR 40 MHz"
- note added: "REDE RF 2,4 GHz - VALORES INICIAIS PARA AJUSTE"
- note added: "Reservas C18/C19 DNP. Nao fabricar sem fechar antena, footprints e ensaios."
- note removed: "ANT1 representa a IFA futura: geometria e casamento dependem da PCB e carcaca."
- note removed: "Cristal 40 MHz CL=8 pF: C14/C15=10 pF pressupoe ~3 pF de parasitas."
- note removed: "LNA_IN isolado de 3V3. C16/L3/C17 sao valores iniciais para ajuste de RF."
- moved on the sheet: ANT1, C14, C15, C16, C17, C18, C19, L3, R14, Y1
