File: Empresa-EcoQuali/EC01/outputs/EC01_KiCad_REV0_2/KiCad/05_Expansao_Display.kicad_sch (KiCad schematic)
At the start: 16 parts, among them J2 DISPLAY 8P DNP, J3 SENSOR INTERNO I2C DNP, U4 TCA9534APWR

Commit message: EC01
Connections:
- net LED_A: no longer names the net of D1.1 (A), R21.2
Other:
- note added: "Antes de habilitar saidas, gravar estados seguros no registrador de saida do U4."
- note added: "BIAS DE PARTIDA"
- note added: "DISPLAY - SELECAO DE INTERFACE"
- note added: "I2C: timeout, tentativa de liberar SDA com SCL e reinicializacao; falha persistente exige power-cycle."
- note added: "SPI: R28/R29. I2C: R30/R31. Nunca montar os dois pares. J2/J3 e seletores DNP na base."
- note added: "U4 - I2C 0x38"
- note removed: "Display SPI: R28/R29. Display I2C: R30/R31. Nunca montar ambos os pares."
- note removed: "J2/J3 DNP. Interface 3,3 V para MODULO; nao aciona painel e-paper diretamente."
- note removed: "U4 TCA9534A: endereco I2C de 7 bits 0x38. Inicializa com portas em entrada."
- moved on the sheet: C22, D1, J2, J3, R21, R22, R23, R24, R25, R26, R27, R28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
