File: Empresa-EcoQuali/EC01/outputs/EC01_KiCad_REV0_2/KiCad/06_Sensores_CAN.kicad_sch (KiCad schematic)
At the start: 24 parts, among them Q2 AO3401A, Q3 2N7002, U5 TCAN330DR, U6 USBLC6-2SC6 DIGITAL, U7 USBLC6-2SC6 DIGITAL

Commit message: EC01
Connections:
- net CAN_RX: no longer names the net of R38.1, U5.4 (RXD)
- net CAN_TERM: no longer names the net of JP1.1 (TERM), R42.2
- net CAN_TX: no longer names the net of R37.2, R41.2, U5.1 (TXD)
- net SENS_GATE: no longer names the net of Q2.1 (G), Q3.3 (D), R32.2
- net SENS_PRE: no longer names the net of F2.1, Q2.3 (D)
Other:
- note added: "ALIMENTACAO CHAVEADA"
- note added: "CAN - MONTAGEM ALTERNATIVA"
- note added: "CAN: montar U5/C24/R37-R41 e TVS apropriadas (D2/D3 TBD). R42/JP1 somente em extremidade."
- note added: "OneWire: R33/R34/R35 + U6/U7. I2C: acrescentar R36. CAN: remover R33-R36 e U6/U7."
- note added: "PTC 100mA nao e limitador preciso. GPIOs em alta impedancia antes de desligar VEXT."
- note added: "RJ11 EM PARALELO / PROTECAO"
- note added: "VEXT: verificar queda em Q2, PTC, cabo e conectores. DS18B20 requer >=3,0 V no sensor."
- note removed: "Base OneWire: R33/R34/R35 e U6/U7. I2C: acrescentar R36. Cabos a definir."
- note removed: "CAN usa um TWAI comum. 120R por R42/JP1 somente na extremidade fisica."
- note removed: "CAN: remover R33-R36 e U6/U7; montar U5/C24/R37-R41. TVS D2/D3 pendentes."
- note removed: "Com VEXT desligada, colocar GPIO1/20 em alta impedancia para evitar realimentacao."
- note removed: "RJ1/RJ2 compartilham barramento. Pinagem LOGICA 1=VEXT 2=GND 3=A 4=B."
- note removed: "VEXT 3,3 V nominal; orcamento 100 mA total. PTC nao e limitador preciso."
- moved on the sheet: C23, C24, D2, D3, F2, JP1, Q2, Q3, R32, R33, R34, R35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
