File: Empresa-EcoQuali/EC01/outputs/EC01_KiCad_REV0_2/KiCad/07_USB_Servico.kicad_sch (KiCad schematic)
At the start: 4 parts, among them J4 USB SERVICE 4P, U8 USBLC6-2SC6

Commit message: EC01
Other:
- note added: "ESD PROXIMO AO CONECTOR NA PCB"
- note added: "ESP32-C3 -> RESISTORES SERIE -> CONECTOR DE SERVICO"
- note added: "J4: 1=GND, 2=D-, 3=D+, 4=NC. Nao e USB-C e nao recebe VBUS/5V."
- note added: "Os 22R ficam proximos ao MCU. U8 fica proximo ao conector, com retorno curto de ESD."
- note added: "Programar com bateria ligada. D-/D+ sao GPIO18/GPIO19; verificar polaridade do cabo."
- note removed: "Gravar com bateria ligada. D-/D+ por R43/R44 e ESD U8."
- note removed: "J4 e header de servico, nao USB-C. Pino 4 NC. Nunca conectar 5 V a 3V3."
- note removed: "USB Serial/JTAG nativo: GPIO18 D- e GPIO19 D+. Verificar cabo e polaridade."
- moved on the sheet: J4, R43, R44, U8
