File: Empresa-EcoQuali/EC01/outputs/EC01_KiCad_REV0_2/KiCad/EC01.kicad_sch (KiCad schematic)
At the start: 0 parts

Commit message: EC01
Other:
- note added: "Consultar ../REVISAO_METODO_EC01.md e BOM para decisoes, limites e pendencias."
- note added: "Duplo clique abre a folha. Rotulos globais ligam folhas; locais ligam blocos na mesma folha."
- note added: "Esquematico nativo KiCad | REV 0.2-R1 | 04 outubro 2026"
- note removed: "Consultar EC01_Documento_de_Engenharia.pdf e BOM para decisoes, limites e pendencias."
- note removed: "Duplo clique em cada folha para abrir o circuito. Redes com o mesmo nome sao globais."
- note removed: "Esquematico nativo KiCad | REV 0.2 | 04 outubro 2026"
